File: ptschematic.sch (EAGLE design)
At the start: 38 parts, among them IC1 7824DT, J3 FEMALE 2x3, U1 ATMEGA328P-AU, Y1 16MHz, Y2 32MHz

Commit message: made changes to lbr and sch
Parts:
- removed C1: 0.1uF, adafruit:C-USC0805
- removed C10, C4, C7, C8: 0.1uF, cap-master:CNP-0805
- removed C2, C3: 22pF, cap-master:CNP-0805
- removed C5, C6, C9: 4.7uF, adafruit:C-USC0805
- removed CN1: (no value), adafruit:USBMINIB
- removed D1: (no value), adafruit:DIODESOD-123
- removed IC1: 7824DT, adafruit:7824DT
- removed LED1, LED2, LED3, LED4: (no value), adafruit:LEDCHIPLED_0805
- removed R3: 100, adafruit:R-US_R0805
- removed R4, R5, R6, R7: 680, adafruit:R-US_R0805
- removed SW1: (no value), adafruit:SWITCH_PUSHBUTTONEVQ-PE
- removed U1: ATMEGA328P-AU, Atmel-ATMEGA328P-AU:ATMEGA328P-AU
- removed U2: (no value), microbuilder:FT232RLSSOP28
- removed Y1: 16MHz, SparkFun-Clocks:CRYSTAL-16MHZPTH-HC49US
- added C16, C17: 10 uF, adafruit:C-USC0805
- added J1: (no value), SparkFun-Connectors:CONN_04X2
- added J2: (no value), SparkFun-Connectors:CONN_02
- added LED5, LED6: (no value), adafruit:LEDCHIPLED_0805
- added R10, R9: 680, adafruit:R-US_R0805
- added TP1, TP2, TP3, TP4: TEST-POINT2, SparkFun-Connectors:TEST-POINT2
- added U3: NCP1117LPST33T3G, NCP1117LPST33T3G:NCP1117LPST33T3G
- added U4: BGM13S, BMES-Spr2019:BGM13S
- added VR1, VR2: 5k, SparkFun-Resistors:TRIMPOT-SMD-5MM-CLOSED-1/4W-20%
- J3: value FEMALE 2x3 -> (none); device SparkFun-Connectors:CONN_03X2FEMALE -> SparkFun-Connectors:CONN_04
- R1: value 680 -> 0
- R2: value 100 -> 0
Connections:
- removed net 3.3V: C7.2, U2.3V3OUT
- removed net A0: U1.PC0
- removed net A1: U1.PC1
- removed net A2: U1.PC2
- removed net A3: U1.PC3
- removed net A4: U1.PC4
- removed net A5: U1.PC5
- removed net A6: U1.ADC6
- removed net A7: U1.ADC7
- removed net AREF: C4.1, U1.AREF
- removed net D0/RX: R2.1, U2.TXD
- removed net D1/TX: R3.1, U2.RXD
- removed net D10: U1.PB2
- removed net D11/MOSI: J3.4, U1.PB3
- removed net D12/MISO: J3.1, U1.PB4
- removed net D13/SCK: J3.3, R4.2, U1.PB5
- removed net D2: U1.PD2
- removed net D3: U1.PD3
- removed net D4: U1.PD4
- removed net D5: U1.PD5
- removed net D6: U1.PD6
- removed net D7: U1.PD7
- removed net D8: U1.PB0
- removed net D9: U1.PB1
- removed net N$12: R6.1, U2.RXLED
- removed net N$13: R7.1, U2.TXLED
- removed net N$14: C8.1, U2.DTR
- removed net N$15: LED4.C, R7.2
- removed net N$7: R2.2, U1.PD0
- removed net N$8: R3.2, U1.PD1
- removed net N$9: LED3.C, R6.2
- removed net RESET: C8.2, J3.5, R1.1, SW1.P$1, U1.PC6
- removed net VUSB: C10.2, C9.1, CN1.VBUS, D1.A
- new net A1RXD: U$1.P2.5, U4.PA0
- new net A1TXD: U$1.P2.6, U4.PA1
- new net ADC1: U$1.P1.2, VR1.WIPER
- new net ADC2: U$1.P1.3, VR2.WIPER
- new net BGMRST: U$1.P3.1, U4.RESETN
- new net N$17: R10.1, U$1.P3.0
- new net N$18: LED6.A, R10.2
- new net RST: J1.3, R8.1, SW2.P$1, U$1.RST
- new net TCK: J1.8, U$1.P1.4
- new net TDI: J1.4, U$1.P1.6
- new net TDO/TDI: J1.2, U$1.P1.7
- new net TEST: J1.5, U$1.TEST
- new net TMS: J1.6, U$1.P1.5
- net +5V: now also C17.1, J1.1, R9.2, TP1.1, TP2.1, U3.OUTPUT, U4.IOVDD, U4.VBATT, VR1.CCW, VR2.CCW; no longer C1.1, C5.1, C6.1, D1.C, IC1.VO, LED3.A, LED4.A, R1.2, R5.2, U1.AVCC, U1.VCC, U1.VCC_2, U2.VCC, U2.VCCIO
- net GND: now also C16.2, C17.2, J1.7, J2.2, LED5.C, LED6.C, R2.2, TP3.1, TP4.1, U3.GND, U4.VSS@1, U4.VSS@10, U4.VSS@11, U4.VSS@2, U4.VSS@3, U4.VSS@4, U4.VSS@5, U4.VSS@6, U4.VSS@7, U4.VSS@8, U4.VSS@9, VR1.CW, VR2.CW; no longer C1.2, C10.1, C2.1, C3.1, C4.2, C5.2, C6.2, C7.1, C9.2, CN1.GND, IC1.GND, J3.6, LED1.C, LED2.C, SW1.P$2, U1.GND, U1.GND_2, U1.GND_3, U2.AGND, U2.GND1, U2.GND2, U2.GND3
- net N$1: now also J3.4, U4.PF0; no longer C3.2, U1.PB7, Y1.2
- net N$10: now also LED5.A, R9.1; no longer R8.1, SW2.P$1, U$1.RST
- net N$2: now also J3.3, U4.PF1; no longer C2.2, U1.PB6, Y1.1
- net N$3: now also J3.2, U4.PF2; no longer LED1.A, R4.1
- net N$4: now also J3.1, U4.PF3; no longer LED2.A, R5.1
- net N$5: now also R1.2, U4.ANTENNA; no longer CN1.D+, U2.USB+
- net N$6: now also R1.1, R2.1, U4.RF; no longer CN1.D-, U2.USB-
- net VIN: now also C16.1, J2.1, U3.INPUT; no longer IC1.VI, J3.2
Other:
- note added: "*note A0 is TX on BGM, but for connection purposes label must be the same"
- moved on the sheet: C11, C12, C13, C14, C15, R1, R2, R8, SW2, Y2
