File: ptschematic.sch (EAGLE design)
At the start: 28 parts, among them U3 NCP1117LPST33T3G, U4 BGM13S, Y2 32MHz

Commit message: finished tracing BGM
Parts:
- removed R1, R2: 0, adafruit:R-US_R0805
Connections:
- removed net N$5: R1.2, U4.ANTENNA
- removed net N$6: R1.1, R2.1, U4.RF
- net ADC1: now also TP4.1
- net ADC2: now also TP3.1
- net GND: now also U4.ANTENNA, U4.ANT_GND, U4.RF; no longer R2.2, TP3.1, TP4.1
Other:
- moved on the sheet: TP3, TP4
Changed lines of the file:
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@@
 <part name="J3" library="SparkFun-Connectors" library_urn="urn:adsk.eagle:library:513" deviceset="CONN_04" device="" package3d_urn="urn:adsk.eagle:package:38085/1"/>
 <part name="GND1" library="supply" deviceset="GND" device=""/>
-<part name="R1" library="adafruit" deviceset="R-US_" device="R0805" value="0"/>
-<part name="R2" library="adafruit" deviceset="R-US_" device="R0805" value="0"/>
 <part name="SUPPLY1" library="SparkFun-PowerSymbols" library_urn="urn:adsk.eagle:library:530" deviceset="3.3V" device=""/>
 <part name="SUPPLY2" library="SparkFun-PowerSymbols" library_urn="urn:adsk.eagle:library:530" deviceset="3.3V" device=""/>
@@
 <part name="SUPPLY7" library="SparkFun-PowerSymbols" library_urn="urn:adsk.eagle:library:530" deviceset="3.3V" device=""/>
 <part name="SUPPLY8" library="SparkFun-PowerSymbols" library_urn="urn:adsk.eagle:library:530" deviceset="3.3V" device=""/>
+<part name="GND2" library="supply" deviceset="GND" device=""/>
 </parts>
 <sheets>
@@
 <instance part="TP1" gate="G$1" x="20.32" y="104.14"/>
 <instance part="TP2" gate="G$1" x="48.26" y="104.14"/>
-<instance part="TP3" gate="G$1" x="48.26" y="88.9"/>
-<instance part="TP4" gate="G$1" x="20.32" y="88.9"/>
+<instance part="TP3" gate="G$1" x="45.72" y="88.9" rot="R270"/>
+<instance part="TP4" gate="G$1" x="20.32" y="88.9" rot="R270"/>
 <instance part="U4" gate="G$1" x="233.68" y="134.62"/>
 <instance part="GND27" gate="1" x="246.38" y="83.82"/>
 <instance part="J3" gate="G$1" x="190.5" y="124.46"/>
 <instance part="GND1" gate="1" x="254" y="172.72"/>
-<instance part="R1" gate="G$1" x="236.22" y="185.42" rot="R270"/>
-<instance part="R2" gate="G$1" x="254" y="185.42" rot="R270"/>
 <instance part="SUPPLY1" gate="G$1" x="83.82" y="205.74"/>
 <instance part="SUPPLY2" gate="G$1" x="83.82" y="205.74"/>
@@
 <instance part="SUPPLY7" gate="G$1" x="226.06" y="180.34"/>
 <instance part="SUPPLY8" gate="G$1" x="231.14" y="180.34"/>
+<instance part="GND2" gate="1" x="246.38" y="175.26"/>
 </instances>
 <busses>
@@
 <pinref part="VR1" gate="R?" pin="CW"/>
 <pinref part="GND24" gate="1" pin="GND"/>
-<wire x1="12.7" y1="91.44" x2="12.7" y2="88.9" width="0.1524" layer="91"/>
-<pinref part="TP4" gate="G$1" pin="1"/>
-<wire x1="12.7" y1="88.9" x2="12.7" y2="86.36" width="0.1524" layer="91"/>
-<wire x1="20.32" y1="88.9" x2="12.7" y2="88.9" width="0.1524" layer="91"/>
-<junction x="12.7" y="88.9"/>
+<wire x1="12.7" y1="91.44" x2="12.7" y2="86.36" width="0.1524" layer="91"/>
 </segment>
 <segment>
 <pinref part="VR2" gate="R?" pin="CW"/>
 <pinref part="GND25" gate="1" pin="GND"/>
-<wire x1="38.1" y1="91.44" x2="38.1" y2="88.9" width="0.1524" layer="91"/>
-<pinref part="TP3" gate="G$1" pin="1"/>
-<wire x1="38.1" y1="88.9" x2="38.1" y2="86.36" width="0.1524" layer="91"/>
-<wire x1="48.26" y1="88.9" x2="38.1" y2="88.9" width="0.1524" layer="91"/>
-<junction x="38.1" y="88.9"/>
+<wire x1="38.1" y1="91.44" x2="38.1" y2="86.36" width="0.1524" layer="91"/>
 </segment>
 <segment>
@@
 </segment>
 <segment>
-<pinref part="R2" gate="G$1" pin="2"/>
 <pinref part="GND1" gate="1" pin="GND"/>
-<wire x1="254" y1="180.34" x2="254" y2="175.26" width="0.1524" layer="91"/>
+<wire x1="236.22" y1="193.04" x2="238.76" y2="193.04" width="0.1524" layer="91"/>
+<wire x1="238.76" y1="193.04" x2="254" y2="193.04" width="0.1524" layer="91"/>
+<pinref part="U4" gate="G$1" pin="RF"/>
+<wire x1="238.76" y1="175.26" x2="238.76" y2="193.04" width="0.1524" layer="91"/>
+<junction x="238.76" y="193.04"/>
+<pinref part="U4" gate="G$1" pin="ANTENNA"/>
+<wire x1="236.22" y1="193.04" x2="236.22" y2="175.26" width="0.1524" layer="91"/>
+<wire x1="254" y1="193.04" x2="254" y2="175.26" width="0.1524" layer="91"/>
+</segment>
+<segment>
+<pinref part="U4" gate="G$1" pin="ANT_GND"/>
+<wire x1="241.3" y1="175.26" x2="241.3" y2="180.34" width="0.1524" layer="91"/>
+<wire x1="241.3" y1="180.34" x2="246.38" y2="180.34" width="0.1524" layer="91"/>
+<wire x1="246.38" y1="180.34" x2="246.38" y2="177.8" width="0.1524" layer="91"/>
+<pinref part="GND2" gate="1" pin="GND"/>
 </segment>
 </net>
@@
 <pinref part="VR1" gate="R?" pin="WIPER"/>
 <wire x1="17.78" y1="96.52" x2="20.32" y2="96.52" width="0.1524" layer="91"/>
-<label x="20.32" y="96.52" size="1.27" layer="95" xref="yes"/>
+<label x="25.4" y="96.52" size="1.27" layer="95" xref="yes"/>
+<pinref part="TP4" gate="G$1" pin="1"/>
+<wire x1="20.32" y1="96.52" x2="25.4" y2="96.52" width="0.1524" layer="91"/>
+<wire x1="20.32" y1="88.9" x2="20.32" y2="96.52" width="0.1524" layer="91"/>
+<junction x="20.32" y="96.52"/>
 </segment>
 <segment>
@@
 <pinref part="VR2" gate="R?" pin="WIPER"/>
 <wire x1="43.18" y1="96.52" x2="45.72" y2="96.52" width="0.1524" layer="91"/>
-<label x="45.72" y="96.52" size="1.27" layer="95" xref="yes"/>
+<label x="50.8" y="96.52" size="1.27" layer="95" xref="yes"/>
+<pinref part="TP3" gate="G$1" pin="1"/>
+<wire x1="45.72" y1="96.52" x2="50.8" y2="96.52" width="0.1524" layer="91"/>
+<wire x1="45.72" y1="88.9" x2="45.72" y2="96.52" width="0.1524" layer="91"/>
+<junction x="45.72" y="96.52"/>
 </segment>
 <segment>
@@
 </segment>
 </net>
-<net name="N$5" class="0">
-<segment>
-<pinref part="R1" gate="G$1" pin="2"/>
-<pinref part="U4" gate="G$1" pin="ANTENNA"/>
-<wire x1="236.22" y1="180.34" x2="236.22" y2="175.26" width="0.1524" layer="91"/>
-</segment>
-</net>
-<net name="N$6" class="0">
-<segment>
-<pinref part="U4" gate="G$1" pin="RF"/>
-<wire x1="238.76" y1="175.26" x2="241.3" y2="175.26" width="0.1524" layer="91"/>
-<wire x1="241.3" y1="175.26" x2="241.3" y2="193.04" width="0.1524" layer="91"/>
-<wire x1="241.3" y1="193.04" x2="254" y2="193.04" width="0.1524" layer="91"/>
-<pinref part="R2" gate="G$1" pin="1"/>
-<wire x1="254" y1="193.04" x2="254" y2="190.5" width="0.1524" layer="91"/>
-<pinref part="R1" gate="G$1" pin="1"/>
-<wire x1="236.22" y1="190.5" x2="236.22" y2="193.04" width="0.1524" layer="91"/>
-<wire x1="236.22" y1="193.04" x2="241.3" y2="193.04" width="0.1524" layer="91"/>
-<junction x="241.3" y="193.04"/>
-</segment>
-</net>

Commit message: updated board and schematic
Connections:
- net 3.3V: now also U$1.P1.0
- net ADC1: now also U$1.P1.1; no longer U$1.P1.2
- net GND: now also U$1.P1.2
Changed lines of the file:
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@@
 <part name="SUPPLY8" library="SparkFun-PowerSymbols" library_urn="urn:adsk.eagle:library:530" deviceset="3.3V" device=""/>
 <part name="GND2" library="supply" deviceset="GND" device=""/>
+<part name="GND3" library="supply" deviceset="GND" device=""/>
+<part name="SUPPLY9" library="SparkFun-PowerSymbols" library_urn="urn:adsk.eagle:library:530" deviceset="3.3V" device=""/>
 </parts>
 <sheets>
@@
 <instance part="SUPPLY8" gate="G$1" x="231.14" y="180.34"/>
 <instance part="GND2" gate="1" x="246.38" y="175.26"/>
+<instance part="GND3" gate="1" x="91.44" y="116.84"/>
+<instance part="SUPPLY9" gate="G$1" x="91.44" y="132.08"/>
 </instances>
 <busses>
@@
 <pinref part="GND2" gate="1" pin="GND"/>
 </segment>
+<segment>
+<pinref part="GND3" gate="1" pin="GND"/>
+<wire x1="91.44" y1="119.38" x2="91.44" y2="121.92" width="0.1524" layer="91"/>
+<pinref part="U$1" gate="G$1" pin="P1.2"/>
+<wire x1="91.44" y1="121.92" x2="114.3" y2="121.92" width="0.1524" layer="91"/>
+</segment>
 </net>
 <net name="VIN" class="0">
@@
 </segment>
 <segment>
-<pinref part="U$1" gate="G$1" pin="P1.2"/>
-<wire x1="114.3" y1="121.92" x2="111.76" y2="121.92" width="0.1524" layer="91"/>
-<label x="111.76" y="121.92" size="1.27" layer="95" rot="R180" xref="yes"/>
+<pinref part="U$1" gate="G$1" pin="P1.1"/>
+<wire x1="114.3" y1="124.46" x2="111.76" y2="124.46" width="0.1524" layer="91"/>
+<label x="111.76" y="124.46" size="1.27" layer="95" rot="R180" xref="yes"/>
 </segment>
 </net>
@@
 <pinref part="SUPPLY7" gate="G$1" pin="3.3V"/>
 </segment>
-</net>
+<segment>
+<pinref part="SUPPLY9" gate="G$1" pin="3.3V"/>
+<wire x1="91.44" y1="132.08" x2="91.44" y2="129.54" width="0.1524" layer="91"/>
+<pinref part="U$1" gate="G$1" pin="P1.0"/>
+<wire x1="91.44" y1="129.54" x2="114.3" y2="129.54" width="0.1524" layer="91"/>
+</segment>
+</net>
